File: kicad/bidirectional_load_switch.kicad_pcb (KiCad board)
At the start: 2 copper layers, 128 parts, among them J101 Screw_Terminal_01x13, U1001 LM25184NGUR, U1002 750313445, U201 SN74LVC1G17DCKR, U202 UCC23313DWYR, U203 SISS94DN-T1-GE3, U204 SISS94DN-T1-GE3, U301 SN74LVC1G17DCKR, U302 UCC23313DWYR, U303 SISS94DN-T1-GE3, U304 SISS94DN-T1-GE3, U401 SN74LVC1G17DCKR, U402 UCC23313DWYR, U403 SISS94DN-T1-GE3, U404 SISS94DN-T1-GE3, U501 SN74LVC1G17DCKR, U502 UCC23313DWYR, U503 SISS94DN-T1-GE3, U504 SISS94DN-T1-GE3, U601 SN74LVC1G17DCKR, U602 UCC23313DWYR, U603 SISS94DN-T1-GE3, U604 SISS94DN-T1-GE3, U701 SN74LVC1G17DCKR, U702 UCC23313DWYR, U703 SISS94DN-T1-GE3, U704 SISS94DN-T1-GE3, U801 SN74LVC1G17DCKR, U802 UCC23313DWYR, U803 SISS94DN-T1-GE3, U804 SISS94DN-T1-GE3, U901 SN74LVC1G17DCKR, U902 UCC23313DWYR, U903 SISS94DN-T1-GE3, U904 SISS94DN-T1-GE3

Commit message: kicad
Parts:
- removed the U901 at (79.9, 56.6)
- added J102: Screw_Terminal_01x02, TerminalBlock:TerminalBlock_Xinya_XY308-2.54-2P_1x02_P2.54mm_Horizontal, F.Cu at (124.2, 34.9)
- added J103: Screw_Terminal_01x09, TerminalBlock:TerminalBlock_Xinya_XY308-2.54-9P_1x09_P2.54mm_Horizontal, F.Cu at (32.0, 104.1)
- added U901: SN74LVC1G17DCKR, buffer_SN74LVC1G17DCKR:DCK5, F.Cu at (79.7, 161.5)
- added U901: SN74LVC1G17DCKR, buffer_SN74LVC1G17DCKR:DCK5, F.Cu at (95.0, 47.5)
- C201, C301, C401, C501, C601, C701, C801, C901: footprint Capacitor_SMD:C_0402_1005Metric -> Capacitor_SMD:C_0603_1608Metric
- J101: value Screw_Terminal_01x13 -> Screw_Terminal_01x03; footprint TerminalBlock:TerminalBlock_Xinya_XY308-2.54-13P_1x13_P2.54mm_Horizontal -> TerminalBlock:TerminalBlock_Xinya_XY308-2.54-3P_1x03_P2.54mm_Horizontal
- moved C201 137.8 mm to (25.5, 156.7)
- moved R201 125.7 mm to (25.2, 158.9)
- moved R202 125.7 mm to (25.2, 160.9)
- moved C203 123.4 mm to (26.4, 153.8)
- moved U202 123.4 mm to (30.6, 148.9)
- moved U203 123.4 mm to (32.2, 154.6)
- moved U204 123.4 mm to (32.2, 159.5)
- moved R203 123.4 mm to (36.8, 157.1)
- moved R204 123.4 mm to (36.8, 159.7)
- moved U201 123.4 mm to (37.1, 154.0)
- moved C202 121.5 mm to (39.1, 146.6)
- moved C204 121.5 mm to (39.1, 148.6)
- moved RS108 96.0 mm to (126.0, 45.0), turned to 180 degrees
- moved C501 82.8 mm to (73.8, 127.5)
- moved C601 82.8 mm to (54.8, 145.8)
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Connections:
- J101 pad 2: 3v3 -> GND
- J101 pad 3: GND -> 3v3
Routing:
- net GNDPWR: track 0.00 -> 13.4 mm, vias 0 -> 12
- net /Channel 8/RIN: track 0.00 -> 7.58 mm
- net GND: track 0.00 -> 7.27 mm, vias 0 -> 8
- net Net-(U902-VOUT): track 0.00 -> 5.12 mm
- net Net-(U904-G): track 0.00 -> 4.56 mm
- net Earth: track 0.00 -> 4.05 mm, vias 0 -> 4
- net 15V_isolated: track 0.00 -> 3.70 mm
- net 3v3: track 0.00 -> 3.17 mm
- net Net-(U901-Y): track 0.00 -> 3.09 mm
- net Net-(U903-G): track 0.00 -> 2.87 mm
- net Net-(U902-ANODE): track 0.00 -> 2.63 mm
- net Net-(U902-CATHODE): track 0.00 -> 2.63 mm
- added copper zone on F.Cu, net /AC_in
- added copper zone on B.Cu, net Earth
- added copper zone on B.Cu, net GND
- added copper zone on B.Cu, net GNDPWR

Commit message: pcb
Parts:
- added U902: UCC23313DWYR, gate_driver_UCC23313DWYR:SOIC6_DWY_TEX, F.Cu at (6.57, 2.72)
- moved R903 0.20 mm to (116.5, 46.7)
- moved R904 0.10 mm to (116.5, 48.4)
Routing:
- net GNDPWR: track 13.4 -> 4.06 mm, vias 12 -> 10
- net /Channel 8/RIN: track 7.58 -> 0.00 mm
- net Net-(U904-G): track 4.56 -> 0.00 mm
- net Earth: track 4.05 -> 0.00 mm, vias 4 -> 8
- net Net-(U903-G): track 2.87 -> 0.00 mm
- added copper zone on F.Cu, net /Channel 8/RIN
- added copper zone on F.Cu, net Earth
- added copper zone on F.Cu, net GNDPWR

Commit message: kicad
Parts:
- removed the U902 at (107.5, 47.5)
- C204, C304, C404, C504, C604, C704, C804, C904: footprint Capacitor_SMD:C_0402_1005Metric -> Capacitor_SMD:C_0805_2012Metric
- RS101, RS102, RS103, RS104, RS105, RS106, RS107, RS108: footprint Resistor_SMD:R_1206_3216Metric_Pad1.30x1.75mm_HandSolder -> Resistor_SMD:R_2512_6332Metric
- moved R201 244.6 mm to (242.2, 46.2)
- moved R202 244.6 mm to (242.2, 48.2)
- moved C201 233.6 mm to (238.3, 60.1)
- moved C203 231.3 mm to (234.8, 53.3)
- moved U202 226.4 mm to (233.5, 48.5)
- moved C202 224.7 mm to (242.0, 50.2)
- moved U201 223.8 mm to (238.7, 56.9)
- moved R601 223.4 mm to (261.6, 64.6)
- moved R602 223.4 mm to (261.6, 66.6)
- moved C204 222.2 mm to (239.8, 53.2)
- moved R203 221.6 mm to (234.1, 56.3)
- moved R204 221.6 mm to (234.1, 58.8)
- moved U203 221.3 mm to (229.5, 54.1)
- moved U204 221.3 mm to (229.5, 59.1)
- moved C601 213.8 mm to (257.7, 78.4)
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Routing:
- net GND: track 7.27 -> 0.00 mm, vias 8 -> 9
- net Net-(U902-VOUT): track 5.12 -> 0.00 mm
- net GNDPWR: track 4.06 -> 0.00 mm, vias 10 -> 20
- net 15V_isolated: track 3.70 -> 0.00 mm, vias 0 -> 6
- net 3v3: track 3.17 -> 0.00 mm
- net Net-(U901-Y): track 3.09 -> 0.00 mm
- net Net-(U902-ANODE): track 2.63 -> 0.00 mm
- net Net-(U902-CATHODE): track 2.63 -> 0.00 mm
- added copper zone on B.Cu, net 15V_isolated
- added copper zone on F.Cu, net 15V_isolated
- added copper zone on F.Cu, net 3v3
- added copper zone on F.Cu, net GND
- added copper zone on F.Cu, net Net-(U901-Y)
- added copper zone on F.Cu, net Net-(U902-ANODE)
- added copper zone on F.Cu, net Net-(U902-CATHODE)
- added copper zone on F.Cu, net Net-(U902-VOUT)
- added copper zone on F.Cu, net Net-(U903-G)
- added copper zone on F.Cu, net Net-(U904-G)
Other:
- rule pad_to_mask_clearance: 0 -> 0.0508
