File: kicad/switching_channel.kicad_sch (KiCad schematic)
At the start: 12 parts, among them U201 SN74LVC1G17DCKR, U202 UCC23313DWYR, U203 SISS94DN-T1-GE3, U204 SISS94DN-T1-GE3

Commit message: kicad
Parts:
- C204: footprint Capacitor_SMD:C_0402_1005Metric -> Capacitor_SMD:C_0805_2012Metric
- U201: footprint DCK5 -> buffer_SN74LVC1G17DCKR:DCK5
- U202: footprint SOIC6_DWY_TEX -> gate_driver_UCC23313DWYR:SOIC6_DWY_TEX
- U203, U204: footprint MOSFET_3DN-T1-GE3_VIS -> mosfet_SISS94DN-T1-GE3:MOSFET_3DN-T1-GE3_VIS
Changed lines of the file:
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@@
 			)
 		)
-		(property "Footprint" "MOSFET_3DN-T1-GE3_VIS"
+		(property "Footprint" "mosfet_SISS94DN-T1-GE3:MOSFET_3DN-T1-GE3_VIS"
 			(at 206.248 100.076 0)
 			(effects
@@
 			)
 		)
-		(property "Footprint" "Capacitor_SMD:C_0402_1005Metric"
+		(property "Footprint" "Capacitor_SMD:C_0805_2012Metric"
 			(at 152.4 132.08 0)
 			(effects
@@
 			)
 		)
-		(property "Footprint" "SOIC6_DWY_TEX"
+		(property "Footprint" "gate_driver_UCC23313DWYR:SOIC6_DWY_TEX"
 			(at 134.62 100.33 0)
 			(effects
@@
 			)
 		)
-		(property "Footprint" "MOSFET_3DN-T1-GE3_VIS"
+		(property "Footprint" "mosfet_SISS94DN-T1-GE3:MOSFET_3DN-T1-GE3_VIS"
 			(at 206.248 105.664 0)
 			(effects
@@
 			)
 		)
-		(property "Footprint" "DCK5"
+		(property "Footprint" "buffer_SN74LVC1G17DCKR:DCK5"
 			(at 95.25 97.79 0)
 			(effects
