File: kicad/bidirectional_load_switch/switching_channel.kicad_sch (KiCad schematic)
At the start: 12 parts, among them U201 SN74LVC1G17DCKR, U202 UCC23313DWYR, U203 SISS94DN-T1-GE3, U204 SISS94DN-T1-GE3

Commit message: psu
Parts:
- C204: footprint Capacitor_SMD:C_0805_2012Metric -> Capacitor_SMD:C_0402_1005Metric
Changed lines of the file:
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@@
 			)
 		)
-		(property "Footprint" "Capacitor_SMD:C_0805_2012Metric"
+		(property "Footprint" "Capacitor_SMD:C_0402_1005Metric"
 			(at 152.4 132.08 0)
 			(effects

Commit message: switch
Parts:
- added LED201: B1911PG--20D000514U1930, led_B1911PG--20D000514U1930:LED_B1911PG--20D000514U1930_HVK, symbol led_B1911PG--20D000514U1930:B1911PG--20D000514U1930
- added R201: 150, Resistor_SMD:R_0603_1608Metric, symbol Device:R_US
- C202, C204: footprint Capacitor_SMD:C_0402_1005Metric -> Capacitor_SMD:C_0603_1608Metric
- R202: renamed from R201; footprint Resistor_SMD:R_0402_1005Metric_Pad0.72x0.64mm_HandSolder -> Resistor_SMD:R_0603_1608Metric
- R203: renamed from R202; footprint Resistor_SMD:R_0402_1005Metric_Pad0.72x0.64mm_HandSolder -> Resistor_SMD:R_0603_1608Metric
- R204: renamed from R203; footprint Resistor_SMD:R_0603_1608Metric_Pad0.98x0.95mm_HandSolder -> Resistor_SMD:R_0805_2012Metric
- R205: renamed from R204; footprint Resistor_SMD:R_0603_1608Metric_Pad0.98x0.95mm_HandSolder -> Resistor_SMD:R_0805_2012Metric
Connections:
- net GND: now also R201.2
- net PWM: now also LED201.2
- new net: LED201.1, R201.1
Other:
- moved on the sheet: C201, C202, C203, C204

Commit message: load switch
Connections:
- net 3v3 renamed 3V3
Other:
- moved on the sheet: C201, C202, C203, C204, LED201, R201, R202, R203, R204, R205, U201, U202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

Commit message: kicad
Parts:
- added TP201, TP202, TP203, TP204: TestPoint, TestPoint:TestPoint_Pad_D1.0mm, symbol Connector:TestPoint
Connections:
- net RIN: now also TP204.1
- net VG1: now reaches R204.2, U203.4 (G)
- net VG1: now also TP202.1
- net ANODE: now reaches R202.2, U202.1 (ANODE)
- net VOUT: now reaches R204.1, R205.1, U202.5 (VOUT)
- net VOUT: now also TP201.1
- net VG2: now reaches R205.2, U204.4 (G)
- net VG2: now also TP203.1
- net BOUT: now reaches R202.1, U201.4 (Y)
Other:
- moved on the sheet: C201, C202, C203, C204, LED201, R201, R202, R203, R204, R205, U201, U202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

Commit message: kicad
Parts:
- removed TP201, TP202, TP203, TP204: TestPoint, TestPoint:TestPoint_Pad_D1.0mm, symbol Connector:TestPoint
