File: kicad/bidirectional_load_switch/switching_channel.kicad_sch (KiCad schematic)
At the start: 14 parts

Commit message: implementing 5v and 3v3 supply ORing
Other:
- title: (none) -> Bidirectional Load Switch
Changed lines of the file:
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@@
 	(paper "A4")
 	(title_block
-		(date "2024-09-17")
-		(rev "0.1.0")
+		(title "Bidirectional Load Switch")
+		(date "2024-10-29")
+		(rev "0.2.0")
 		(company "University of Wisconsin-Platteville")
 		(comment 1 "Nicholas Loehrke")

Commit message: schematic capture
Changed lines of the file:
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@@
 	(text_box "Bidirectional switch"
 		(exclude_from_sim no)
-		(at 183.515 63.5 0)
-		(size 57.15 70.485)
+		(at 182.88 63.5 0)
+		(size 57.785 70.485)
 		(stroke
 			(width 0)
