File: kicad/bidirectional_load_switch/bidirectional_load_switch.kicad_sch (KiCad schematic)
At the start: 11 parts, among them J101 Screw_Terminal_01x03, J102 Screw_Terminal_01x02, J103 Screw_Terminal_01x09

Commit message: switch
Parts:
- removed J101: Screw_Terminal_01x03, TerminalBlock:TerminalBlock_Xinya_XY308-2.54-3P_1x03_P2.54mm_Horizontal, symbol Connector:Screw_Terminal_01x03
- removed J102: Screw_Terminal_01x02, TerminalBlock:TerminalBlock_Xinya_XY308-2.54-2P_1x02_P2.54mm_Horizontal, symbol Connector:Screw_Terminal_01x02
- removed J103: Screw_Terminal_01x09, TerminalBlock:TerminalBlock_Xinya_XY308-2.54-9P_1x09_P2.54mm_Horizontal, symbol Connector:Screw_Terminal_01x09
- added J101: Conn_01x02_Socket, Connector_PinHeader_2.54mm:PinHeader_1x02_P2.54mm_Vertical, symbol Connector:Conn_01x02_Socket
- added J102: 282838-2, CONN2_282838-2_TEC, symbol screw_terminal_282838-2:282838-2
- added J103: Conn_01x09_Socket, Connector_PinHeader_2.54mm:PinHeader_1x09_P2.54mm_Vertical, symbol Connector:Conn_01x09_Socket
Connections:
- net AC_in: now also J102.1
- net Earth: now also J102.2
- net GND: now also J103.9 (Pin_9)
- net PWM1: now also J103.1 (Pin_1)
- net PWM2: now also J103.2 (Pin_2)
- net PWM3: now also J103.3 (Pin_3)
- net PWM4: now also J103.4 (Pin_4)
- net PWM5: now also J103.5 (Pin_5)
- net PWM6: now also J103.6 (Pin_6)
- net PWM7: now also J103.7 (Pin_7)
- net PWM8: now also J103.8 (Pin_8)
- new net 15V_isolated: J101.1 (Pin_1)
- new net GNDPWR: J101.2 (Pin_2)
Other:
- removed sheet Isolated DC-DC
- note removed: "- check gate resistor power rating"

Commit message: load switch
Parts:
- added C101, C104: 100n, Capacitor_SMD:C_0603_1608Metric, symbol Device:C_Small
- added C102, C103: 10u, Capacitor_SMD:C_1206_3216Metric, symbol Device:C_Small
- added J104: Conn_01x02_Socket, Connector_PinHeader_2.54mm:PinHeader_1x02_P2.54mm_Vertical, symbol Connector:Conn_01x02_Socket
- added U101: LDL212PV33R, ldo_LDL212PV33R:DFN_V33R_STM, symbol ldo_LDL212PV33R:LDL212PV33R
- J101: renamed from J102; footprint CONN2_282838-2_TEC -> screw_terminal_282838-2:CONN2_282838-2_TEC
- renumbered J101 to J102
Connections:
- net GND: now also C101.2, C102.2, C103.2, C104.2, J104.2 (Pin_2), U101.1 (GND), U101.7 (GND)
- new net 3V3: C103.1, C104.1, U101.2 (ADJ/sense), U101.3 (VOUT)
- new net 5V: C101.1, C102.1, J104.1 (Pin_1), U101.4 (VIN), U101.6 (EN)
Other:
- moved on the sheet: J101, J102, J103, RS101, RS102, RS103, RS104, RS105, RS106, RS107, RS108

Commit message: kicad
Parts:
- removed J101: 282838-2, screw_terminal_282838-2:CONN2_282838-2_TEC, symbol screw_terminal_282838-2:282838-2
- added J101: 1017503, 1017503:PHOENIX_1017503, symbol spring_terminal_1017503:1017503
- added R101: 120k, symbol Device:R_US
- added R102: 150k, symbol Device:R_US
- added U102: TLV3201AIDCKR, TLV3201AIDCKR:SOT65P210X110-5N, symbol comparator_TLV3201AIDCKR:TLV3201AIDCKR
- added U103: TMCS1101A3BQDR, SOIC8_D_TEX, symbol current_sensor_TMCS1101A3BQDR:TMCS1101A3BQDR
- added U104: SN74LVC2G02DCUR, DCU8_TEX, symbol nor_gate_SN74LVC2G02DCUR:SN74LVC2G02DCUR
- added U105: SN74LVC08APWR, PW14, symbol and_gate_SN74LVC08APWR:SN74LVC08APWR
- RS101: value R_US -> 1
- RS102: value R_US -> 3.9
- RS103: value R_US -> 15
- RS104: value R_US -> 47
- RS105: value R_US -> 200
- RS106: value R_US -> 680
- RS107: value R_US -> 2700
- RS108: value R_US -> 10000
Connections:
- net 3V3: now also R101.1, U102.5 (VCC), U103.8 (VS)
- net AC_in: now also J101.2_1, J101.2_2, U103.1 (IN+), U103.2 (IN+); no longer RS101.1, RS102.1, RS103.1, RS104.1, RS105.1, RS106.1, RS107.1, RS108.1
- net Earth: now also J101.1_1, J101.1_2
- net GND: now also R102.2, U102.2 (GND), U103.5 (GND), U104.4 (GND)
- net PWM1: no longer J103.1 (Pin_1)
- net PWM2: no longer J103.2 (Pin_2)
- net PWM3: no longer J103.3 (Pin_3)
- net PWM4: no longer J103.4 (Pin_4)
- net PWM5: no longer J103.5 (Pin_5)
- net PWM6: no longer J103.6 (Pin_6)
- net PWM7: no longer J103.7 (Pin_7)
- net PWM8: no longer J103.8 (Pin_8)
- new net: U102.3 (IN+), U103.7 (VOUT)
- new net: U104.2 (1B), U104.3 (2Y)
- new net: U104.5 (2A), U104.7 (1Y)
- new net AC_post_sense: RS101.1, RS102.1, RS103.1, RS104.1, RS105.1, RS106.1, RS107.1, RS108.1, U103.3 (IN-), U103.4 (IN-)
- new net PWM1_in: J103.1 (Pin_1), U105.2 (1B)
- new net PWM2_in: J103.2 (Pin_2), U105.5 (2B)
- new net PWM3_in: J103.3 (Pin_3), U105.13 (4B)
- new net PWM4_in: J103.4 (Pin_4), U105.10 (3B)
- new net PWM5_in: J103.5 (Pin_5)
- new net PWM6_in: J103.6 (Pin_6)
- new net PWM7_in: J103.7 (Pin_7)
- new net PWM8_in: J103.8 (Pin_8)
- new net V_{ref}: R101.2, R102.1, U102.4 (IN-)
- new net fault: U102.1 (OUT), U104.6 (2B)
- new net fault_reset: U104.1 (1A)
- new net ~{fault}: U104.8 (VCC), U105.1 (1A), U105.12 (4A), U105.4 (2A), U105.9 (3A)
Other:
- note added: "V_{out} = 0.2I_{in} + 0.5V_{S} For I_{fault} = 1 A and V_{s} = 3.3 V: V_{ref} = 1.85 V"
- moved on the sheet: C101, C102, C103, C104, J102, J103, J104, RS101, RS102, RS103, RS104, RS105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

Commit message: idk
Connections:
- net 3V3: now also U104.8 (VCC)
- net fault: no longer U104.6 (2B)
- net ~{fault}: no longer U104.8 (VCC)
- new net fault_set: U104.6 (2B)
Changed lines of the file:
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@@
 	(wire
 		(pts
-			(xy 220.98 45.72) (xy 234.95 45.72)
+			(xy 220.98 45.72) (xy 233.68 45.72)
 		)
 		(stroke
@@
 	(wire
 		(pts
-			(xy 220.98 43.18) (xy 223.52 43.18)
-		)
-		(stroke
-			(width 0)
-			(type default)
-		)
-	)
-	(wire
-		(pts
 			(xy 184.15 96.52) (xy 190.5 96.52)
 		)
@@
 	(wire
 		(pts
-			(xy 234.95 40.64) (xy 234.95 45.72)
+			(xy 233.68 40.64) (xy 233.68 45.72)
 		)
 		(stroke
@@
 	(wire
 		(pts
-			(xy 220.98 38.1) (xy 223.52 38.1)
-		)
-		(stroke
-			(width 0)
-			(type default)
-		)
-	)
-	(wire
-		(pts
 			(xy 59.69 36.83) (xy 59.69 38.1)
 		)
@@
 	(wire
 		(pts
+			(xy 222.25 35.56) (xy 223.52 35.56)
+		)
+		(stroke
+			(width 0)
+			(type default)
+		)
+	)
+	(wire
+		(pts
 			(xy 138.43 31.75) (xy 139.7 31.75)
 		)
@@
 	(wire
 		(pts
-			(xy 220.98 40.64) (xy 234.95 40.64)
+			(xy 220.98 40.64) (xy 233.68 40.64)
 		)
 		(stroke
@@
 	(wire
 		(pts
+			(xy 222.25 35.56) (xy 222.25 38.1)
+		)
+		(stroke
+			(width 0)
+			(type default)
+		)
+	)
+	(wire
+		(pts
 			(xy 80.01 38.1) (xy 80.01 39.37)
 		)
@@
 		(pts
 			(xy 118.11 134.62) (xy 127 134.62)
+		)
+		(stroke
+			(width 0)
+			(type default)
+		)
+	)
+	(wire
+		(pts
+			(xy 222.25 38.1) (xy 220.98 38.1)
+		)
+		(stroke
+			(width 0)
+			(type default)
+		)
+	)
+	(wire
+		(pts
+			(xy 220.98 43.18) (xy 222.25 43.18)
 		)
 		(stroke
@@
 		)
 	)
-	(label "~{fault}"
-		(at 223.52 38.1 0)
-		(fields_autoplaced yes)
-		(effects
-			(font
-				(size 1.27 1.27)
-			)
-			(justify left bottom)
-		)
-	)
 	(label "PWM4_in"
 		(at 102.87 139.7 180)
@@
 		)
 	)
-	(label "fault"
-		(at 223.52 43.18 0)
-		(fields_autoplaced yes)
-		(effects
-			(font
-				(size 1.27 1.27)
-			)
-			(justify left bottom)
-		)
-	)
 	(label "fault_reset"
 		(at 187.96 38.1 0)
@@
 	(label "AC_post_sense"
 		(at 64.77 43.18 0)
+		(fields_autoplaced yes)
+		(effects
+			(font
+				(size 1.27 1.27)
+			)
+			(justify left bottom)
+		)
+	)
+	(label "fault_set"
+		(at 222.25 43.18 0)
 		(fields_autoplaced yes)
 		(effects
@@
 				(hide yes)
 			)
+		)
+	)
+	(global_label "3V3"
+		(shape input)
+		(at 223.52 35.56 0)
+		(fields_autoplaced yes)
+		(effects
+			(font
+				(size 1.27 1.27)
+			)
+			(justify left)
+		)
+		(property "Intersheetrefs" "${INTERSHEET_REFS}"
+			(at 230.0128 35.56 0)
+			(effects
+				(font
+					(size 1.27 1.27)
+				)
+				(justify left)
+				(hide yes)
+			)

Commit message: idk
Connections:
- net fault_set is gone; now on net fault: U104.6 (2B)
Changed lines of the file:
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@@
 		)
 	)
-	(label "fault_set"
+	(label "fault"
 		(at 222.25 43.18 0)
 		(fields_autoplaced yes)

Commit message: idk
Parts:
- removed R101: 120k, symbol Device:R_US
- removed R102: 150k, symbol Device:R_US
- removed U102: TLV3201AIDCKR, TLV3201AIDCKR:SOT65P210X110-5N, symbol comparator_TLV3201AIDCKR:TLV3201AIDCKR
- removed U104: SN74LVC2G02DCUR, DCU8_TEX, symbol nor_gate_SN74LVC2G02DCUR:SN74LVC2G02DCUR
Other:
- note removed: "V_{out} = 0.2I_{in} + 0.5V_{S} For I_{fault} = 1 A and V_{s} = 3.3 V: V_{ref} = 1.85 V"

Commit message: i hate layouts
Parts:
- removed U105: SN74LVC08APWR, PW14, symbol and_gate_SN74LVC08APWR:SN74LVC08APWR
- added C101, C104, C109: 100n, Capacitor_SMD:C_0603_1608Metric, symbol Device:C_Small
- added J105, J106: Conn_01x02_Socket, Connector_PinHeader_2.54mm:PinHeader_1x02_P2.54mm_Vertical, symbol Connector:Conn_01x02_Socket
- added J107: AVR-ISP-6, Connector_IDC:IDC-Header_2x03_P2.54mm_Vertical, symbol isp:AVR-ISP-6
- added R101, R102: 10k, Resistor_SMD:R_0603_1608Metric, symbol Device:R_US
- added SW101: PTS526 SK15 SMTR2 LFS, switch_switch_PTS526_SK15_SMTR2_LFS:SMT_FS, symbol switch_PTS526_SK15_SMTR2_LFS:PTS526_SK15_SMTR2_LFS
- added U104: ATTINY85-20SU, mcu_ATTINY85_20SU:8S2_ATM, symbol mcu_ATTINY85-20SU:ATTINY85-20SU
- J101: footprint 1017503:PHOENIX_1017503 -> spring_terminal_1017503:PHOENIX_1017503
- U101: renamed from U103; footprint SOIC8_D_TEX -> current_sensor_TMCS1101A3BQDR:SOIC8_D_TEX
- renumbered C101 to C105, C102 to C106, C103 to C107, C104 to C108, J103 to J102, J104 to J103, J102 to J104, U101 to U105
Connections:
- net 3V3: now also C101.1, C104.1, J107.2 (VCC), R102.1, U104.8 (VCC)
- net 5V: now also J103.2 (Pin_2); no longer J103.1 (Pin_1)
- net AC_in: now also U101.3 (IN-), U101.4 (IN-); no longer U101.1 (IN+), U101.2 (IN+)
- net AC_post_sense: now also U101.1 (IN+), U101.2 (IN+); no longer U101.3 (IN-), U101.4 (IN-)
- net GND: now also J103.1 (Pin_1), C101.2, C104.2, C109.2, J105.2 (Pin_2), J106.2 (Pin_2), J107.6 (GND), SW101.1, SW101.2, U104.4 (GND); no longer J103.2 (Pin_2)
- net ~{fault}: now also U104.3 (PB4)
- net at U101.7 (VOUT): now also R101.1
- new net: R101.2, U104.2 (PB3)
- new net MISO/fault_status: J105.1 (Pin_1), J107.1 (MISO), U104.6 (PB1)
- new net MOSI: J107.4 (MOSI), U104.5 (PB0)
- new net SCK/~{fault_rst}: J106.1 (Pin_1), J107.3 (SCK), U104.7 (PB2)
- new net ~{MCU_RST}: C109.1, J107.5 (~{RST}), R102.2, SW101.3, SW101.4, U104.1 (PB5)
Other:
- note added: "15 volt isolated input"
- note added: "5 volt input w/3V3 regulator"
- note added: "AC input w/overcurrent protection"
- note added: "ISP programmer header"
- note added: "MCU"
- note added: "MCU reset button"
- note added: "PB connector for overcurrent fault reset"
- note added: "Switching channels"
- note added: "current sensor"
- note added: "digital output for overcurrent fault status"
- moved on the sheet: C105, C106, C107, C108, J101, J102, J103, J104, RS101, RS102, RS103, RS104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

Commit message: :|
Parts:
- removed U105: LDL212PV33R, ldo_LDL212PV33R:DFN_V33R_STM, symbol ldo_LDL212PV33R:LDL212PV33R
- added U102: TLV75733PDBVR, DBV0005A_N, symbol ldo_TLV75733PDBVR:TLV75733PDBVR
Connections:
- net 3V3: now also U102.4 (NC), U102.5 (OUT)
- net 5V: now also U102.1 (IN), U102.3 (EN)
- net GND: now also U102.2 (GND)
Other:
- moved on the sheet: C107, C108
