File: kicad/power_supply/isolated_dc_to_dc.kicad_sch (KiCad schematic)
At the start: 23 parts, among them U1001 LM25184NGUR, U1002 750313445

Commit message: psu
Other:
- moved on the sheet: C1001, C1002, C1003, C1004, C1005, C1006, C1007, C1008, C_{SNB}1001, Css1001, D_{C}1001, D_{FLY}1001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

Commit message: kicad
Parts:
- renumbered C1001 to C201, C1002 to C202, C1003 to C203, C1004 to C204, C1005 to C205, C1006 to C206, C1007 to C207, C1008 to C208, C_{SNB}1001 to C_{SNB}201, Css1001 to Css201, D_{C}1001 to D_{C}201, D_{FLY}1001 to D_{FLY}201, D_{F}1001 to D_{F}201, D_{Z}1001 to D_{Z}201, R_{DUMMY}1001 to R_{DUMMY}201, R_{FB}1001 to R_{FB}201, R_{SET}1001 to R_{SET}201, R_{SNB}1001 to R_{SNB}201, Rtc1001 to Rtc201, Ruv1001 to Ruv201, Ruv1002 to Ruv202, U1001 to U201, U1002 to U202
Changed lines of the file:
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@@
 		(on_board yes)
 		(dnp no)
-		(property "Reference" "Ruv1001"
+		(property "Reference" "Ruv201"
 			(at 73.152 110.49 0)
 			(effects
@@
 			(project ""
 				(path "/a4768a02-c961-4971-939f-bbf2bfa51fa3/64dc0b5a-21d5-4edc-b6c2-a4fad2cceb53"
-					(reference "Ruv1001")
+					(reference "Ruv201")
 					(unit 1)
 				)
@@
 		(on_board yes)
 		(dnp yes)
-		(property "Reference" "R_{SNB}1001"
+		(property "Reference" "R_{SNB}201"
 			(at 173.228 55.88 90)
 			(effects
@@
 			(project ""
 				(path "/a4768a02-c961-4971-939f-bbf2bfa51fa3/64dc0b5a-21d5-4edc-b6c2-a4fad2cceb53"
-					(reference "R_{SNB}1001")
+					(reference "R_{SNB}201")
 					(unit 1)
 				)
@@
 		(on_board yes)
 		(dnp yes)
-		(property "Reference" "D_{Z}1001"
+		(property "Reference" "D_{Z}201"
 			(at 210.82 75.692 90)
 			(effects
@@
 			(project "bidirectional_load_switch"
 				(path "/a4768a02-c961-4971-939f-bbf2bfa51fa3/64dc0b5a-21d5-4edc-b6c2-a4fad2cceb53"
-					(reference "D_{Z}1001")
+					(reference "D_{Z}201")
 					(unit 1)
 				)
@@
 		(on_board yes)
 		(dnp no)
-		(property "Reference" "C1002"
+		(property "Reference" "C202"
 			(at 163.322 116.332 0)
 			(effects
@@
 			(project "bidirectional_load_switch"
 				(path "/a4768a02-c961-4971-939f-bbf2bfa51fa3/64dc0b5a-21d5-4edc-b6c2-a4fad2cceb53"
-					(reference "C1002")
+					(reference "C202")
 					(unit 1)
 				)
@@
 		(dnp no)
 		(fields_autoplaced yes)
-		(property "Reference" "#PWR01005"
+		(property "Reference" "#PWR0205"
 			(at 200.66 129.54 0)
 			(effects
@@
 			(project "bidirectional_load_switch"
 				(path "/a4768a02-c961-4971-939f-bbf2bfa51fa3/64dc0b5a-21d5-4edc-b6c2-a4fad2cceb53"
-					(reference "#PWR01005")
+					(reference "#PWR0205")
 					(unit 1)
 				)
@@
 		(on_board yes)
 		(dnp no)
-		(property "Reference" "C1008"
+		(property "Reference" "C208"
 			(at 216.916 116.332 0)
 			(effects
@@
 			(project "bidirectional_load_switch"
 				(path "/a4768a02-c961-4971-939f-bbf2bfa51fa3/64dc0b5a-21d5-4edc-b6c2-a4fad2cceb53"
-					(reference "C1008")
+					(reference "C208")
 					(unit 1)
 				)
@@
 		(on_board yes)
 		(dnp no)
-		(property "Reference" "C1005"
+		(property "Reference" "C205"
 			(at 193.802 116.332 0)
 			(effects
@@
 			(project "bidirectional_load_switch"
 				(path "/a4768a02-c961-4971-939f-bbf2bfa51fa3/64dc0b5a-21d5-4edc-b6c2-a4fad2cceb53"
-					(reference "C1005")
+					(reference "C205")
 					(unit 1)
 				)
@@
 		(on_board yes)
 		(dnp no)
-		(property "Reference" "R_{FB}1001"
+		(property "Reference" "R_{FB}201"
 			(at 135.89 100.076 0)
 			(effects
@@
 			(project "bidirectional_load_switch"
 				(path "/a4768a02-c961-4971-939f-bbf2bfa51fa3/64dc0b5a-21d5-4edc-b6c2-a4fad2cceb53"
-					(reference "R_{FB}1001")
+					(reference "R_{FB}201")
 					(unit 1)
 				)
@@
 		(on_board yes)
 		(dnp no)
-		(property "Reference" "C1001"
+		(property "Reference" "C201"
 			(at 155.702 116.332 0)
 			(effects
@@
 			(project ""
 				(path "/a4768a02-c961-4971-939f-bbf2bfa51fa3/64dc0b5a-21d5-4edc-b6c2-a4fad2cceb53"
-					(reference "C1001")
+					(reference "C201")
 					(unit 1)
 				)
@@
 		(on_board yes)
 		(dnp no)
-		(property "Reference" "C1006"
+		(property "Reference" "C206"
 			(at 201.422 116.332 0)
 			(effects
@@
 			(project "bidirectional_load_switch"
 				(path "/a4768a02-c961-4971-939f-bbf2bfa51fa3/64dc0b5a-21d5-4edc-b6c2-a4fad2cceb53"
-					(reference "C1006")
+					(reference "C206")
 					(unit 1)
 				)
@@
 		(on_board yes)
 		(dnp no)
-		(property "Reference" "C1007"
+		(property "Reference" "C207"
 			(at 209.042 116.332 0)
 			(effects
@@
 			(project "bidirectional_load_switch"
 				(path "/a4768a02-c961-4971-939f-bbf2bfa51fa3/64dc0b5a-21d5-4edc-b6c2-a4fad2cceb53"
-					(reference "C1007")
+					(reference "C207")
 					(unit 1)
 				)
@@
 		(on_board yes)
 		(dnp no)
-		(property "Reference" "D_{FLY}1001"
+		(property "Reference" "D_{FLY}201"
 			(at 180.34 66.294 0)
 			(effects
@@
 			(project "bidirectional_load_switch"
 				(path "/a4768a02-c961-4971-939f-bbf2bfa51fa3/64dc0b5a-21d5-4edc-b6c2-a4fad2cceb53"
-					(reference "D_{FLY}1001")
+					(reference "D_{FLY}201")
 					(unit 1)
 				)
@@
 		(on_board yes)
 		(dnp yes)
-		(property "Reference" "R_{DUMMY}1001"
+		(property "Reference" "R_{DUMMY}201"
 			(at 188.468 75.438 0)
 			(effects
@@
 			(project "bidirectional_load_switch"
 				(path "/a4768a02-c961-4971-939f-bbf2bfa51fa3/64dc0b5a-21d5-4edc-b6c2-a4fad2cceb53"
-					(reference "R_{DUMMY}1001")
+					(reference "R_{DUMMY}201")
 					(unit 1)
 				)
@@
 		(on_board yes)
 		(dnp no)
-		(property "Reference" "C1003"
+		(property "Reference" "C203"
 			(at 171.196 116.332 0)
 			(effects
@@
 			(project "bidirectional_load_switch"
 				(path "/a4768a02-c961-4971-939f-bbf2bfa51fa3/64dc0b5a-21d5-4edc-b6c2-a4fad2cceb53"
-					(reference "C1003")
+					(reference "C203")
 					(unit 1)
 				)
@@
 		(on_board yes)
 		(dnp no)
-		(property "Reference" "Rtc1001"
+		(property "Reference" "Rtc201"
 			(at 85.598 110.49 0)
 			(effects
@@
 			(project "bidirectional_load_switch"
 				(path "/a4768a02-c961-4971-939f-bbf2bfa51fa3/64dc0b5a-21d5-4edc-b6c2-a4fad2cceb53"
-					(reference "Rtc1001")
+					(reference "Rtc201")
 					(unit 1)
 				)
@@
 		(dnp no)
 		(fields_autoplaced yes)
-		(property "Reference" "#PWR01004"
+		(property "Reference" "#PWR0204"
 			(at 198.12 97.79 0)
 			(effects
@@
 			(project "bidirectional_load_switch"
 				(path "/a4768a02-c961-4971-939f-bbf2bfa51fa3/64dc0b5a-21d5-4edc-b6c2-a4fad2cceb53"
-					(reference "#PWR01004")
+					(reference "#PWR0204")
 					(unit 1)
 				)
@@
 		(on_board yes)
 		(dnp yes)
-		(property "Reference" "C_{SNB}1001"
+		(property "Reference" "C_{SNB}201"
 			(at 183.642 55.88 90)
 			(effects
@@
 			(project "bidirectional_load_switch"
 				(path "/a4768a02-c961-4971-939f-bbf2bfa51fa3/64dc0b5a-21d5-4edc-b6c2-a4fad2cceb53"
-					(reference "C_{SNB}1001")
+					(reference "C_{SNB}201")
 					(unit 1)
 				)
@@
 		(on_board yes)
 		(dnp no)
-		(property "Reference" "R_{SET}1001"
+		(property "Reference" "R_{SET}201"
 			(at 85.598 120.65 0)
 			(effects
@@
 			(project "bidirectional_load_switch"
 				(path "/a4768a02-c961-4971-939f-bbf2bfa51fa3/64dc0b5a-21d5-4edc-b6c2-a4fad2cceb53"
-					(reference "R_{SET}1001")
+					(reference "R_{SET}201")
 					(unit 1)
 				)
@@
 		(on_board yes)
 		(dnp no)
-		(property "Reference" "D_{F}1001"
+		(property "Reference" "D_{F}201"
 			(at 128.016 89.154 90)
 			(effects
@@
 			(project ""
 				(path "/a4768a02-c961-4971-939f-bbf2bfa51fa3/64dc0b5a-21d5-4edc-b6c2-a4fad2cceb53"
-					(reference "D_{F}1001")
+					(reference "D_{F}201")
 					(unit 1)
 				)
@@
 		(dnp no)
 		(fields_autoplaced yes)
-		(property "Reference" "#PWR01003"
+		(property "Reference" "#PWR0203"
 			(at 162.56 130.81 0)
 			(effects
@@
 			(project "bidirectional_load_switch"
 				(path "/a4768a02-c961-4971-939f-bbf2bfa51fa3/64dc0b5a-21d5-4edc-b6c2-a4fad2cceb53"
-					(reference "#PWR01003")
+					(reference "#PWR0203")
 					(unit 1)
 				)
@@
 		(dnp no)
 		(fields_autoplaced yes)
-		(property "Reference" "#PWR01002"
+		(property "Reference" "#PWR0202"
 			(at 134.62 129.54 0)
 			(effects
@@
 			(project ""
 				(path "/a4768a02-c961-4971-939f-bbf2bfa51fa3/64dc0b5a-21d5-4edc-b6c2-a4fad2cceb53"
-					(reference "#PWR01002")
+					(reference "#PWR0202")
 					(unit 1)
 				)
@@
 		(on_board yes)
 		(dnp no)
-		(property "Reference" "Ruv1002"
+		(property "Reference" "Ruv202"
 			(at 73.152 120.65 0)
 			(effects
@@
 			(project ""
 				(path "/a4768a02-c961-4971-939f-bbf2bfa51fa3/64dc0b5a-21d5-4edc-b6c2-a4fad2cceb53"
-					(reference "Ruv1002")
+					(reference "Ruv202")
 					(unit 1)
 				)
@@
 		(on_board yes)
 		(dnp no)
-		(property "Reference" "D_{C}1001"
+		(property "Reference" "D_{C}201"
 			(at 127.762 80.264 90)
 			(effects
@@
 			(project ""
 				(path "/a4768a02-c961-4971-939f-bbf2bfa51fa3/64dc0b5a-21d5-4edc-b6c2-a4fad2cceb53"
-					(reference "D_{C}1001")
+					(reference "D_{C}201")
 					(unit 1)
 				)
@@
 		(dnp no)
 		(fields_autoplaced yes)
-		(property "Reference" "Css1001"
+		(property "Reference" "Css201"
 			(at 137.16 113.0362 0)
 			(effects
@@
 			(project ""
 				(path "/a4768a02-c961-4971-939f-bbf2bfa51fa3/64dc0b5a-21d5-4edc-b6c2-a4fad2cceb53"
-					(reference "Css1001")
+					(reference "Css201")
 					(unit 1)
 				)
@@
 		(dnp no)
 		(fields_autoplaced yes)
-		(property "Reference" "U1002"
+		(property "Reference" "U202"
 			(at 154.305 63.5 0)
 			(effects
@@
 			(project ""
 				(path "/a4768a02-c961-4971-939f-bbf2bfa51fa3/64dc0b5a-21d5-4edc-b6c2-a4fad2cceb53"
-					(reference "U1002")
+					(reference "U202")
 					(unit 1)
 				)
@@
 		(on_board yes)
 		(dnp no)
-		(property "Reference" "C1004"
+		(property "Reference" "C204"
 			(at 186.182 116.332 0)
 			(effects
@@
 			(project "bidirectional_load_switch"
 				(path "/a4768a02-c961-4971-939f-bbf2bfa51fa3/64dc0b5a-21d5-4edc-b6c2-a4fad2cceb53"
-					(reference "C1004")
+					(reference "C204")
 					(unit 1)
 				)
@@
 		(dnp no)
 		(fields_autoplaced yes)
-		(property "Reference" "#PWR01001"
+		(property "Reference" "#PWR0201"
 			(at 82.55 137.16 0)
 			(effects
@@
 			(project ""
 				(path "/a4768a02-c961-4971-939f-bbf2bfa51fa3/64dc0b5a-21d5-4edc-b6c2-a4fad2cceb53"
-					(reference "#PWR01001")
+					(reference "#PWR0201")
 					(unit 1)
 				)
@@
 		(dnp no)
 		(fields_autoplaced yes)
-		(property "Reference" "U1001"
+		(property "Reference" "U201"
 			(at 114.3 86.36 0)
 			(effects
@@
 			(project ""
 				(path "/a4768a02-c961-4971-939f-bbf2bfa51fa3/64dc0b5a-21d5-4edc-b6c2-a4fad2cceb53"
-					(reference "U1001")
-					(unit 1)
-				)
+					(reference "U201")
+					(unit 1)
+				)

Commit message: updated psu
Parts:
- added C209: 100n, Capacitor_SMD:C_0402_1005Metric, symbol Device:C_Small
- C203, C208: value 100n -> 10u; footprint Capacitor_SMD:C_0402_1005Metric -> Capacitor_SMD:C_1206_3216Metric
- C204: value 10u -> 100n; footprint Capacitor_SMD:C_1206_3216Metric -> Capacitor_SMD:C_0402_1005Metric
- R_{FB}201: value 196k -> 75k
- Rtc201: value 787k -> 300k
Connections:
- net 15V_isolated: now also C209.1; no longer C204.1
- net GND: now also C204.2
- net GNDPWR: now also C209.2; no longer C204.2
- net VBAT_managed: now also C204.1
Other:
- note added: "9-25 Vdc"
- note added: "isolated"
- note added: "p_{max}: 0.3W"
- note added: "v_{max}: 98V"
- note removed: "+"
- note removed: "-"
- note removed: "9-13 Vdc"
- moved on the sheet: C_{SNB}201, Css201, D_{C}201, D_{FLY}201, D_{F}201, D_{Z}201, R_{DUMMY}201, R_{FB}201, R_{SET}201, R_{SNB}201, Rtc201, Ruv201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
