File: kicad/power_supply/power_supply.kicad_pcb (KiCad board)
At the start: 2 copper layers, 130 parts, among them J101 Screw_Terminal_01x03, J102 Screw_Terminal_01x02, J103 Screw_Terminal_01x09, U1001 LM25184NGUR, U1002 750313445, U201 SN74LVC1G17DCKR, U202 UCC23313DWYR, U203 SISS94DN-T1-GE3, U204 SISS94DN-T1-GE3, U301 SN74LVC1G17DCKR, U302 UCC23313DWYR, U303 SISS94DN-T1-GE3, U304 SISS94DN-T1-GE3, U401 SN74LVC1G17DCKR, U402 UCC23313DWYR, U403 SISS94DN-T1-GE3, U404 SISS94DN-T1-GE3, U501 SN74LVC1G17DCKR, U502 UCC23313DWYR, U503 SISS94DN-T1-GE3, U504 SISS94DN-T1-GE3, U601 SN74LVC1G17DCKR, U602 UCC23313DWYR, U603 SISS94DN-T1-GE3, U604 SISS94DN-T1-GE3, U701 SN74LVC1G17DCKR, U702 UCC23313DWYR, U703 SISS94DN-T1-GE3, U704 SISS94DN-T1-GE3, U801 SN74LVC1G17DCKR, U802 UCC23313DWYR, U803 SISS94DN-T1-GE3, U804 SISS94DN-T1-GE3, U901 SN74LVC1G17DCKR, U902 UCC23313DWYR, U903 SISS94DN-T1-GE3, U904 SISS94DN-T1-GE3

Commit message: updated psu
Parts:
- removed C1001, C1002, C1004, C1005, C1006, C1007, C303, C403, C503, C603, C703, C803, C903: 10u, Capacitor_SMD:C_1206_3216Metric
- removed C1003, C1008, C302, C304, C402, C404, C502, C504, C602, C604, C702, C704, C802, C804, C902, C904, Css1001: 100n, Capacitor_SMD:C_0402_1005Metric
- removed C301, C401, C501, C601, C701, C801, C901: 1u, Capacitor_SMD:C_0603_1608Metric
- removed C_{SNB}1001: 22p, Capacitor_SMD:C_0402_1005Metric
- removed D_{C}1001, D_{Z}1001: PDZVTR9.1B, zener_PDZVTR9.1B:DIO_PDZVTFT_ROM
- removed D_{FLY}1001, D_{F}1001: SK510A-LTP, schottky_SK510A-LTP:SMADO-214AC_LEAD-FRAME_MCC
- removed J101: Screw_Terminal_01x03, TerminalBlock:TerminalBlock_Xinya_XY308-2.54-3P_1x03_P2.54mm_Horizontal
- removed J102: Screw_Terminal_01x02, TerminalBlock:TerminalBlock_Xinya_XY308-2.54-2P_1x02_P2.54mm_Horizontal
- removed J103: Screw_Terminal_01x09, TerminalBlock:TerminalBlock_Xinya_XY308-2.54-9P_1x09_P2.54mm_Horizontal
- removed R201, R202, R301, R302, R401, R402, R501, R502, R601, R602, R701, R702, R801, R802, R901, R902: 50, Resistor_SMD:R_0402_1005Metric_Pad0.72x0.64mm_HandSolder
- removed R203, R204, R303, R304, R403, R404, R503, R504, R603, R604, R703, R704, R803, R804, R903, R904: 5, Resistor_SMD:R_0603_1608Metric_Pad0.98x0.95mm_HandSolder
- removed RS101, RS102, RS103, RS104, RS105, RS106, RS107, RS108: R_US, Resistor_SMD:R_2512_6332Metric
- removed R_{DUMMY}1001: 1.5k, Resistor_SMD:R_0402_1005Metric
- removed R_{FB}1001: 196k, Resistor_SMD:R_0402_1005Metric
- removed R_{SET}1001: 12.1k, Resistor_SMD:R_0402_1005Metric
- removed R_{SNB}1001: 100, Resistor_SMD:R_0402_1005Metric
- removed Rtc1001: 787k, Resistor_SMD:R_0402_1005Metric
- removed Ruv1001: 46.4k, Resistor_SMD:R_0402_1005Metric
- removed Ruv1002: 10.7k, Resistor_SMD:R_0402_1005Metric
- removed U1001: LM25184NGUR, dc_to_dc_LM25184NGUR:NGU0008C-IPC_A
- removed U1002: 750313445, transformer_750313445:SOIC_13445_WRE
- removed U203, U204, U303, U304, U403, U404, U503, U504, U603, U604, U703, U704, U803, U804, U903, U904: SISS94DN-T1-GE3, mosfet_SISS94DN-T1-GE3:MOSFET_3DN-T1-GE3_VIS
- removed U301, U401, U501, U601, U701, U801, U901: SN74LVC1G17DCKR, buffer_SN74LVC1G17DCKR:DCK5
- removed U302, U402, U502, U602, U702, U802, U902: UCC23313DWYR, gate_driver_UCC23313DWYR:SOIC6_DWY_TEX
- added C205: 10u, Capacitor_SMD:C_1206_3216Metric, F.Cu at (81.9, 78.8)
- added C206: 10u, Capacitor_SMD:C_1206_3216Metric, F.Cu at (81.9, 82.2)
- added C207: 10u, Capacitor_SMD:C_1206_3216Metric, F.Cu at (81.9, 85.5)
- added C208: 100n, Capacitor_SMD:C_0402_1005Metric, F.Cu at (80.5, 88.2)
- added C_{SNB}201: 22p, Capacitor_SMD:C_0402_1005Metric, F.Cu at (80.5, 90.2)
- added Css201: 100n, Capacitor_SMD:C_0402_1005Metric, F.Cu at (80.5, 92.1)
- added D_{C}201: PDZVTR9.1B, zener_PDZVTR9.1B:DIO_PDZVTFT_ROM, F.Cu at (88.2, 88.4)
- added D_{FLY}201: SK510A-LTP, schottky_SK510A-LTP:SMADO-214AC_LEAD-FRAME_MCC, F.Cu at (88.7, 79.5)
- added D_{F}201: SK510A-LTP, schottky_SK510A-LTP:SMADO-214AC_LEAD-FRAME_MCC, F.Cu at (88.7, 84.0)
- added D_{Z}201: PDZVTR9.1B, zener_PDZVTR9.1B:DIO_PDZVTFT_ROM, F.Cu at (88.2, 92.5)
- added R_{DUMMY}201: 1.5k, Resistor_SMD:R_0402_1005Metric, F.Cu at (77.6, 78.2)
- added R_{FB}201: 196k, Resistor_SMD:R_0402_1005Metric, F.Cu at (77.6, 80.2)
- added R_{SET}201: 12.1k, Resistor_SMD:R_0402_1005Metric, F.Cu at (77.6, 82.1)
- added R_{SNB}201: 100, Resistor_SMD:R_0402_1005Metric, F.Cu at (77.6, 84.1)
- added Rtc201: 787k, Resistor_SMD:R_0402_1005Metric, F.Cu at (77.6, 86.1)
- added Ruv201: 46.4k, Resistor_SMD:R_0402_1005Metric, F.Cu at (77.6, 88.1)
- added Ruv202: 10.7k, Resistor_SMD:R_0402_1005Metric, F.Cu at (77.6, 90.1)
- C201: value 1u -> 10u; footprint Capacitor_SMD:C_0603_1608Metric -> Capacitor_SMD:C_1206_3216Metric
- C202, C204: value 100n -> 10u; footprint Capacitor_SMD:C_0402_1005Metric -> Capacitor_SMD:C_1206_3216Metric
- C203: value 10u -> 100n; footprint Capacitor_SMD:C_1206_3216Metric -> Capacitor_SMD:C_0402_1005Metric
- U201: value SN74LVC1G17DCKR -> LM25184NGUR; footprint buffer_SN74LVC1G17DCKR:DCK5 -> dc_to_dc_LM25184NGUR:NGU0008C-IPC_A
- U202: value UCC23313DWYR -> 750313445; footprint gate_driver_UCC23313DWYR:SOIC6_DWY_TEX -> transformer_750313445:SOIC_13445_WRE
- moved U202 10.1 mm to (114.9, 40.4)
- moved U201 1.62 mm to (128.2, 53.0)
Connections:
- C201 pad 1: 3v3 -> VBAT_managed
- C202 pad 1: 3v3 -> VBAT_managed
- C203 pad 1: 15V_isolated -> VBAT_managed
- C203 pad 2: GNDPWR -> GND
- U201 pad 1: unconnected-(U201-NC-Pad1) -> Net-(U201-SW)
- U201 pad 2: /PWM1 -> Net-(U201-FB)
- U201 pad 3: GND -> VBAT_managed
- U201 pad 5: 3v3 -> Net-(U201-SS_BIAS)
- U202 pad 1: Net-(U202-ANODE) -> unconnected-(U202-Pad1)
- U202 pad 2: unconnected-(U202-NC-Pad2) -> Net-(U201-SW)
- U202 pad 3: Net-(U202-CATHODE) -> unconnected-(U202-Pad3)
- U202 pad 4: GNDPWR -> VBAT_managed
- U202 pad 5: Net-(U202-VOUT) -> Net-(D_{FLY}201-Pad2)
- U202 pad 6: 15V_isolated -> Net-(D_{FLY}201-Pad2)

Commit message: updated psu
Parts:
- added C209: 100n, Capacitor_SMD:C_0402_1005Metric, F.Cu at (137.7, 69.9)
- C203, C208: value 100n -> 10u; footprint Capacitor_SMD:C_0402_1005Metric -> Capacitor_SMD:C_1206_3216Metric
- C204: value 10u -> 100n; footprint Capacitor_SMD:C_1206_3216Metric -> Capacitor_SMD:C_0402_1005Metric
- R_{FB}201: value 196k -> 75k
- Rtc201: value 787k -> 300k
Connections:
- C204 pad 1: 15V_isolated -> VBAT_managed
- C204 pad 2: GNDPWR -> GND
