File: kicad/power_supply/power_supply.kicad_sch (KiCad schematic)
At the start: 0 parts

Commit message: psu
Other:
- added sheet 5 Volt DC-DC (5_volt_dc_to_dc.kicad_sch)
Changed lines of the file:
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@@
 	)
 	(sheet
-		(at 85.09 53.34)
+		(at 59.69 48.26)
 		(size 19.05 21.59)
 		(fields_autoplaced yes)
@@
 		)
 		(property "Sheetname" "Isolated DC-DC"
-			(at 85.09 52.6284 0)
+			(at 59.69 47.5484 0)
 			(effects
 				(font
@@
 		)
 		(property "Sheetfile" "isolated_dc_to_dc.kicad_sch"
-			(at 85.09 75.5146 0)
+			(at 59.69 70.4346 0)
 			(effects
 				(font
@@
 			(project "power_supply"
 				(path "/a4768a02-c961-4971-939f-bbf2bfa51fa3"
-					(page "1")
+					(page "2")
 				)
 			)
+		)
+	)
+	(sheet
+		(at 142.24 60.96)
+		(size 25.4 21.59)
+		(fields_autoplaced yes)
+		(stroke
+			(width 0.1524)
+			(type solid)
+		)
+		(fill
+			(color 0 0 0 0.0000)
+		)
+		(property "Sheetname" "5 Volt DC-DC"
+			(at 142.24 60.2484 0)
+			(effects
+				(font
+					(size 1.27 1.27)
+				)
+				(justify left bottom)
+			)
+		)
+		(property "Sheetfile" "5_volt_dc_to_dc.kicad_sch"
+			(at 142.24 83.1346 0)
+			(effects
+				(font
+					(size 1.27 1.27)
+				)
+				(justify left top)
+			)
+		)
+		(instances
+			(project "power_supply"
+				(path "/a4768a02-c961-4971-939f-bbf2bfa51fa3"
+					(page "3")
+				)
+			)

Commit message: kicad
Other:
- sheet Isolated DC-DC renamed 15 Volt Isolated DC-DC
Changed lines of the file:
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@@
 	(sheet
 		(at 59.69 48.26)
-		(size 19.05 21.59)
+		(size 24.13 21.59)
 		(fields_autoplaced yes)
 		(stroke
@@
 			(color 0 0 0 0.0000)
 		)
-		(property "Sheetname" "Isolated DC-DC"
+		(property "Sheetname" "15 Volt Isolated DC-DC"
 			(at 59.69 47.5484 0)
 			(effects
@@
 				)
 				(justify left top)
+				(hide yes)
 			)
 		)
@@
 	)
 	(sheet
-		(at 142.24 60.96)
-		(size 25.4 21.59)
+		(at 109.22 48.26)
+		(size 24.13 21.59)
 		(fields_autoplaced yes)
 		(stroke
@@
 		)
 		(property "Sheetname" "5 Volt DC-DC"
-			(at 142.24 60.2484 0)
+			(at 109.22 47.5484 0)
 			(effects
 				(font
@@
 		)
 		(property "Sheetfile" "5_volt_dc_to_dc.kicad_sch"
-			(at 142.24 83.1346 0)
+			(at 109.22 70.4346 0)
 			(effects
 				(font
@@
 				)
 				(justify left top)
+				(hide yes)
 			)
 		)

Commit message: updated psu
Changed lines of the file:
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@@
 	)
 	(sheet
-		(at 59.69 48.26)
+		(at 67.945 48.26)
 		(size 24.13 21.59)
 		(fields_autoplaced yes)
@@
 		)
 		(property "Sheetname" "15 Volt Isolated DC-DC"
-			(at 59.69 47.5484 0)
+			(at 67.945 47.5484 0)
 			(effects
 				(font
@@
 		)
 		(property "Sheetfile" "isolated_dc_to_dc.kicad_sch"
-			(at 59.69 70.4346 0)
+			(at 67.945 70.4346 0)
 			(effects
 				(font
