File: boards/power_supply/pcb/usb_c_pd.kicad_sch (KiCad schematic)
At the start: 46 parts, among them J201 Conn_01x04_Socket, J202 12401826E412A, J203 USB IDC, SW201 PTS526 SK15 SMTR2 LFS, U201 USBLC6-2P6

Commit message: starting psu layout
Parts:
- C201, C202, C203, C204, C205, C206: footprint (none) -> Capacitor_SMD:C_0603_1608Metric
- J201: footprint (none) -> Connector_PinHeader_2.54mm:PinHeader_1x04_P2.54mm_Vertical
- J202: footprint (none) -> 12401826E412A:12401826E412A
- J203: footprint (none) -> Connector_PinHeader_2.54mm:PinHeader_1x05_P2.54mm_Vertical
- JP201, JP202, JP203: footprint (none) -> Jumper:SolderJumper-2_P1.3mm_Bridged_RoundedPad1.0x1.5mm
- R201, R202, R203, R204, R205, R206, R207, R208, R209, R210, R211, R212, R213, R214, R215, R216, R217: footprint (none) -> Resistor_SMD:R_0603_1608Metric
- SW201: footprint SMT_FS -> PTS526_SK15_SMTR2_LFS:SMT_FS
- TP201, TP202, TP203, TP204, TP205, TP206: footprint (none) -> TestPoint:TestPoint_Pad_D1.0mm
- U203, U204: footprint (none) -> SISA35DN-T1-GE3:SISA35DN-T1-GE3
Changed lines of the file:
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@@
 			)
 		)
-		(property "Footprint" ""
+		(property "Footprint" "Capacitor_SMD:C_0603_1608Metric"
 			(at 204.47 64.77 0)
 			(effects
@@
 			)
 		)
-		(property "Footprint" ""
+		(property "Footprint" "Capacitor_SMD:C_0603_1608Metric"
 			(at 58.42 72.39 0)
 			(effects
@@
 			)
 		)
-		(property "Footprint" ""
+		(property "Footprint" "Resistor_SMD:R_0603_1608Metric"
 			(at 55.88 111.76 0)
 			(effects
@@
 			)
 		)
-		(property "Footprint" ""
+		(property "Footprint" "Resistor_SMD:R_0603_1608Metric"
 			(at 67.31 162.56 0)
 			(effects
@@
 			)
 		)
-		(property "Footprint" ""
+		(property "Footprint" "Capacitor_SMD:C_0603_1608Metric"
 			(at 154.94 64.77 0)
 			(effects
@@
 			)
 		)
-		(property "Footprint" ""
+		(property "Footprint" "SISA35DN-T1-GE3:SISA35DN-T1-GE3"
 			(at 232.41 45.72 0)
 			(effects
@@
 			)
 		)
-		(property "Footprint" ""
+		(property "Footprint" "SISA35DN-T1-GE3:SISA35DN-T1-GE3"
 			(at 220.98 45.72 0)
 			(effects
@@
 			)
 		)
-		(property "Footprint" ""
+		(property "Footprint" "Capacitor_SMD:C_0603_1608Metric"
 			(at 204.47 59.69 0)
 			(effects
@@
 			)
 		)
-		(property "Footprint" ""
+		(property "Footprint" "Resistor_SMD:R_0603_1608Metric"
 			(at 222.25 46.99 0)
 			(effects
@@
 			)
 		)
-		(property "Footprint" ""
+		(property "Footprint" "Resistor_SMD:R_0603_1608Metric"
 			(at 72.39 162.56 0)
 			(effects
@@
 			)
 		)
-		(property "Footprint" ""
+		(property "Footprint" "TestPoint:TestPoint_Pad_D1.0mm"
 			(at 184.15 146.05 0)
 			(effects
@@
 			)
 		)
-		(property "Footprint" ""
+		(property "Footprint" "Connector_PinHeader_2.54mm:PinHeader_1x05_P2.54mm_Vertical"
 			(at 134.62 179.07 0)
 			(effects
@@
 			)
 		)
-		(property "Footprint" ""
+		(property "Footprint" "Resistor_SMD:R_0603_1608Metric"
 			(at 260.35 66.04 0)
 			(effects
@@
 			)
 		)
-		(property "Footprint" ""
+		(property "Footprint" "Connector_PinHeader_2.54mm:PinHeader_1x04_P2.54mm_Vertical"
 			(at 43.18 124.46 0)
 			(effects
@@
 			)
 		)
-		(property "Footprint" ""
+		(property "Footprint" "TestPoint:TestPoint_Pad_D1.0mm"
 			(at 184.15 135.89 0)
 			(effects
@@
 			)
 		)
-		(property "Footprint" "SMT_FS"
+		(property "Footprint" "PTS526_SK15_SMTR2_LFS:SMT_FS"
 			(at 40.132 68.834 0)
 			(effects
@@
 			)
 		)
-		(property "Footprint" ""
+		(property "Footprint" "Jumper:SolderJumper-2_P1.3mm_Bridged_RoundedPad1.0x1.5mm"
 			(at 67.31 173.99 0)
 			(effects
@@
 			)
 		)
-		(property "Footprint" ""
+		(property "Footprint" "Resistor_SMD:R_0603_1608Metric"
 			(at 163.83 135.89 0)
 			(effects
@@
 			)
 		)
-		(property "Footprint" ""
+		(property "Footprint" "Resistor_SMD:R_0603_1608Metric"
 			(at 163.83 140.97 0)
 			(effects
@@
 			)
 		)
-		(property "Footprint" ""
+		(property "Footprint" "Resistor_SMD:R_0603_1608Metric"
 			(at 242.57 52.07 0)
 			(effects
@@
 			)
 		)
-		(property "Footprint" ""
+		(property "Footprint" "TestPoint:TestPoint_Pad_D1.0mm"
 			(at 184.15 140.97 0)
 			(effects
@@
 			)
 		)
-		(property "Footprint" ""
+		(property "Footprint" "Resistor_SMD:R_0603_1608Metric"
 			(at 53.34 72.39 0)
 			(effects
@@
 			)
 		)
-		(property "Footprint" ""
+		(property "Footprint" "Resistor_SMD:R_0603_1608Metric"
 			(at 60.96 111.76 0)
 			(effects
@@
 			)
 		)
-		(property "Footprint" ""
+		(property "Footprint" "Resistor_SMD:R_0603_1608Metric"
 			(at 217.17 58.42 0)
 			(effects
@@
 			)
 		)
-		(property "Footprint" ""
+		(property "Footprint" "TestPoint:TestPoint_Pad_D1.0mm"
 			(at 184.15 161.29 0)
 			(effects
@@
 			)
 		)
-		(property "Footprint" ""
+		(property "Footprint" "Jumper:SolderJumper-2_P1.3mm_Bridged_RoundedPad1.0x1.5mm"
 			(at 72.39 173.99 0)
 			(effects
@@
 			)
 		)
-		(property "Footprint" ""
+		(property "Footprint" "12401826E412A:12401826E412A"
 			(at 123.19 100.33 0)
 			(effects
@@
 			)
 		)
-		(property "Footprint" ""
+		(property "Footprint" "TestPoint:TestPoint_Pad_D1.0mm"
 			(at 184.15 151.13 0)
 			(effects
@@
 			)
 		)
-		(property "Footprint" ""
+		(property "Footprint" "Resistor_SMD:R_0603_1608Metric"
 			(at 163.83 130.81 0)
 			(effects
@@
 			)
 		)
-		(property "Footprint" ""
+		(property "Footprint" "Resistor_SMD:R_0603_1608Metric"
 			(at 163.83 151.13 0)
 			(effects
@@
 			)
 		)
-		(property "Footprint" ""
+		(property "Footprint" "Resistor_SMD:R_0603_1608Metric"
 			(at 163.83 146.05 0)
 			(effects
@@
 			)
 		)
-		(property "Footprint" ""
+		(property "Footprint" "Capacitor_SMD:C_0603_1608Metric"
 			(at 247.65 46.99 0)
 			(effects
@@
 			)
 		)
-		(property "Footprint" ""
+		(property "Footprint" "Capacitor_SMD:C_0603_1608Metric"
 			(at 179.07 57.15 0)
 			(effects
@@
 			)
 		)
-		(property "Footprint" ""
+		(property "Footprint" "Jumper:SolderJumper-2_P1.3mm_Bridged_RoundedPad1.0x1.5mm"
 			(at 58.42 104.14 0)
 			(effects
@@
 			)
 		)
-		(property "Footprint" ""
+		(property "Footprint" "Resistor_SMD:R_0603_1608Metric"
 			(at 160.02 57.15 0)
 			(effects
@@
 			)
 		)
-		(property "Footprint" ""
+		(property "Footprint" "Resistor_SMD:R_0603_1608Metric"
 			(at 163.83 156.21 0)
 			(effects
@@
 			)
 		)
-		(property "Footprint" ""
+		(property "Footprint" "Resistor_SMD:R_0603_1608Metric"
 			(at 160.02 64.77 0)
 			(effects
@@
 			)
 		)
-		(property "Footprint" ""
+		(property "Footprint" "TestPoint:TestPoint_Pad_D1.0mm"
 			(at 184.15 156.21 0)
 			(effects

Commit message: initial psu charger layout
Parts:
- removed J202: 12401826E412A, 12401826E412A:12401826E412A, symbol 12401826E412A:USB_C_Receptacle
- added J202: USB4105-GF-A, USB4105-GF-A:USB4105-GF-A, symbol USB4105-GF-A:USB4105-GF-A
Connections:
- net CC1: now also J202.A5 (CC1)
- net CC2: now also J202.B5 (CC2)
- net GND: now also J202.A1_B12 (GND), J202.B1_A12 (GND)
- net VBUS: now also J202.A4_B9 (VBUS), J202.B4_A9 (VBUS)
- net pre_esd_D_N: now also J202.A7 (D-), J202.B7 (D-)
- net pre_esd_D_P: now also J202.A6 (D+), J202.B6 (D+)
- new net SHIELD: J202.SH1 (SHIELD), J202.SH2 (SHIELD), J202.SH3 (SHIELD), J202.SH4 (SHIELD)
- no-connect marks 13 -> 5
Changed lines of the file:
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@@
 	)
 	(no_connect
-		(at 134.62 123.19)
-	)
-	(no_connect
-		(at 134.62 133.35)
-	)
-	(no_connect
-		(at 134.62 107.95)
-	)
-	(no_connect
-		(at 134.62 118.11)
-	)
-	(no_connect
-		(at 134.62 110.49)
-	)
-	(no_connect
 		(at 134.62 100.33)
 	)
 	(no_connect
-		(at 111.76 140.97)
+		(at 113.03 113.03)
 	)
 	(no_connect
@@
 	)
 	(no_connect
-		(at 134.62 130.81)
-	)
-	(no_connect
-		(at 134.62 115.57)
-	)
-	(no_connect
-		(at 134.62 125.73)
-	)
-	(no_connect
 		(at 134.62 102.87)
 	)
@@
 	(wire
 		(pts
-			(xy 184.15 151.13) (xy 166.37 151.13)
+			(xy 60.96 33.02) (xy 74.93 33.02)
 		)
 		(stroke
@@
 	(wire
 		(pts
-			(xy 90.17 35.56) (xy 85.09 35.56)
+			(xy 184.15 151.13) (xy 166.37 151.13)
 		)
 		(stroke
@@
 	(wire
 		(pts
-			(xy 58.42 68.58) (xy 53.34 68.58)
+			(xy 85.09 35.56) (xy 90.17 35.56)
 		)
 		(stroke
@@
 	(wire
 		(pts
-			(xy 67.31 160.02) (xy 67.31 158.75)
+			(xy 58.42 68.58) (xy 53.34 68.58)
 		)
 		(stroke
@@
 	(wire
 		(pts
-			(xy 72.39 168.91) (xy 72.39 170.18)
+			(xy 67.31 160.02) (xy 67.31 158.75)
 		)
 		(stroke
@@
 	(wire
 		(pts
-			(xy 74.93 33.02) (xy 60.96 33.02)
+			(xy 72.39 168.91) (xy 72.39 170.18)
 		)
 		(stroke
@@
 	(wire
 		(pts
-			(xy 119.38 140.97) (xy 119.38 143.51)
+			(xy 119.38 113.03) (xy 119.38 115.57)
 		)
 		(stroke
@@
 	(wire
 		(pts
-			(xy 60.96 35.56) (xy 74.93 35.56)
-		)
-		(stroke
-			(width 0)
-			(type default)
-		)
-	)
-	(wire
-		(pts
 			(xy 134.62 74.93) (xy 137.16 74.93)
 		)
@@
 	(wire
 		(pts
-			(xy 90.17 33.02) (xy 85.09 33.02)
+			(xy 55.88 114.3) (xy 55.88 119.38)
 		)
 		(stroke
@@
 	(wire
 		(pts
-			(xy 55.88 114.3) (xy 55.88 119.38)
+			(xy 201.93 88.9) (xy 214.63 88.9)
 		)
 		(stroke
@@
 	(wire
 		(pts
-			(xy 201.93 88.9) (xy 214.63 88.9)
+			(xy 36.83 40.64) (xy 40.64 40.64)
 		)
 		(stroke
@@
 	(wire
 		(pts
-			(xy 36.83 40.64) (xy 40.64 40.64)
+			(xy 69.85 156.21) (xy 69.85 158.75)
 		)
 		(stroke
@@
 	(wire
 		(pts
-			(xy 69.85 156.21) (xy 69.85 158.75)
+			(xy 60.96 35.56) (xy 74.93 35.56)
 		)
 		(stroke
@@
 	(wire
 		(pts
+			(xy 85.09 33.02) (xy 90.17 33.02)
+		)
+		(stroke
+			(width 0)
+			(type default)
+		)
+	)
+	(wire
+		(pts
 			(xy 60.96 121.92) (xy 48.26 121.92)
 		)
@@
 		)
 	)
+	(label "VSNK"
+		(at 251.46 43.18 0)
+		(fields_autoplaced yes)
+		(effects
+			(font
+				(size 1.27 1.27)
+			)
+			(justify left bottom)
+		)
+	)
 	(label "ADDR1"
 		(at 163.83 106.68 0)
@@
 	(symbol
 		(lib_id "power:GND")
-		(at 119.38 143.51 0)
+		(at 119.38 115.57 0)
 		(unit 1)
 		(exclude_from_sim no)
@@
 		(fields_autoplaced yes)
 		(property "Reference" "#PWR0206"
-			(at 119.38 149.86 0)
+			(at 119.38 121.92 0)
 			(effects
 				(font
@@
 		)
 		(property "Value" "GND"
-			(at 119.38 148.59 0)
+			(at 119.38 120.65 0)
 			(effects
 				(font
@@
 		)
 		(property "Footprint" ""
-			(at 119.38 143.51 0)
+			(at 119.38 115.57 0)
 			(effects
 				(font
@@
 		)
 		(property "Datasheet" ""
-			(at 119.38 143.51 0)
+			(at 119.38 115.57 0)
 			(effects
 				(font
@@
 		)
 		(property "Description" "Power symbol creates a global label with name \"GND\" , ground"
-			(at 119.38 143.51 0)
+			(at 119.38 115.57 0)
 			(effects
 				(font
@@
 	)
 	(symbol
-		(lib_id "12401826E412A:USB_C_Receptacle")
-		(at 119.38 100.33 0)
-		(unit 1)
-		(exclude_from_sim no)
-		(in_bom yes)
-		(on_board yes)
-		(dnp no)
-		(property "Reference" "J202"
-			(at 119.38 67.31 0)
-			(effects
-				(font
-					(size 1.27 1.27)
-				)
-			)
-		)
-		(property "Value" "12401826E412A"
-			(at 119.38 69.85 0)
-			(effects
-				(font
-					(size 1.27 1.27)
-				)
-				(hide yes)
-			)
-		)
-		(property "Footprint" "12401826E412A:12401826E412A"
-			(at 123.19 100.33 0)
-			(effects
-				(font
-					(size 1.27 1.27)
-				)
-				(hide yes)
-			)
-		)
-		(property "Datasheet" "https://cdn.amphenol-cs.com/media/wysiwyg/files/documentation/datasheet/inputoutput/io_usb_type_c.pdf"
-			(at 123.19 100.33 0)
-			(effects
-				(font
-					(size 1.27 1.27)
-				)
-				(hide yes)
-			)
-		)
-		(property "Description" "CONN RCP USB3.1 TYPEC 24P SMD RA"
-			(at 119.38 100.33 0)
-			(effects
-				(font
-					(size 1.27 1.27)
-				)
-				(hide yes)
-			)
-		)
-		(property "MPN" "12401826E412A"
-			(at 119.38 70.358 0)
-			(effects
-				(font
-					(size 1.27 1.27)
-				)
-			)
-		)
-		(pin "A2"
-		)
-		(pin "A8"
-		)
-		(pin "S1"
-		)
-		(pin "B9"
-		)
-		(pin "A10"
-		)
-		(pin "B3"
-		)
-		(pin "A12"
-		)
-		(pin "B11"
-		)
-		(pin "B1"
-		)
-		(pin "B5"
-		)
-		(pin "A3"
-		)
-		(pin "A6"
-		)
-		(pin "A1"
-		)
-		(pin "B4"
-		)
-		(pin "B12"
-		)
-		(pin "B7"
-		)
-		(pin "A9"
-		)
-		(pin "A7"
-		)
-		(pin "B10"
-		)
-		(pin "B2"
-		)
-		(pin "B6"
-		)
-		(pin "A11"
-		)
-		(pin "A4"
-		)
-		(pin "A5"
-		)
-		(pin "B8"
-		)
-		(instances
-			(project "power_supply"
-				(path "/6a7d9dc9-f78f-470f-911b-b95256023173/4a384965-6a35-4bf6-849e-cb865e62d5b4"
-					(reference "J202")
-					(unit 1)
-				)
-			)
-		)
-	)
-	(symbol
 		(lib_id "Connector:TestPoint")
 		(at 184.15 146.05 270)
@@
 					(unit 1)
 				)
+			)
+		)
+	)
+	(symbol
+		(lib_id "USB4105-GF-A:USB4105-GF-A")
+		(at 134.62 74.93 0)
+		(unit 1)
+		(exclude_from_sim no)
+		(in_bom yes)
+		(on_board yes)
+		(dnp no)
+		(fields_autoplaced yes)
+		(property "Reference" "J202"
+			(at 119.0625 67.31 0)
+			(effects
+				(font
+					(size 1.27 1.27)
+				)
+			)
+		)
+		(property "Value" "USB4105-GF-A"
+			(at 110.998 65.532 0)
+			(effects
+				(font
+					(size 1.27 1.27)
+				)
+				(justify left bottom)
+				(hide yes)
+			)
+		)
+		(property "Footprint" "USB4105-GF-A:USB4105-GF-A"
+			(at 117.856 62.992 0)
+			(effects
+				(font
+					(size 1.27 1.27)
+				)
+				(justify bottom)
+				(hide yes)
+			)
+		)
+		(property "Datasheet" "https://mm.digikey.com/Volume0/opasdata/d220001/medias/docus/5492/USB4105.pdf"
+			(at 118.11 67.31 0)
+			(effects
+				(font
+					(size 1.27 1.27)
+				)
+				(hide yes)
+			)
+		)
+		(property "Description" ""
+			(at 118.745 95.25 0)
+			(effects
+				(font
+					(size 1.27 1.27)
+				)
+				(hide yes)
+			)
+		)
+		(property "MPN" "USB4105-GF-A"
+			(at 119.0625 69.85 0)
+			(effects
+				(font
+					(size 1.27 1.27)
+				)
+			)
+		)
+		(pin "A1_B12"
+		)
+		(pin "B1_A12"
+		)
+		(pin "SH2"
+		)
+		(pin "A8"
+		)
+		(pin "A5"
+		)
+		(pin "SH3"
+		)
+		(pin "A4_B9"
+		)
+		(pin "A6"
+		)
+		(pin "B5"
+		)
+		(pin "B4_A9"
+		)
+		(pin "A7"
+		)
+		(pin "B7"
+		)
+		(pin "SH1"
+		)
+		(pin "B8"
+		)
+		(pin "SH4"
+		)
+		(pin "B6"
+		)
+		(instances
+			(project ""
+				(path "/6a7d9dc9-f78f-470f-911b-b95256023173/4a384965-6a35-4bf6-849e-cb865e62d5b4"
+					(reference "J202")
+					(unit 1)
+				)

Commit message: psu layouting
Connections:
- net VBUS: no longer U203.6, U203.7, U203.8
- net VSNK: no longer U204.6, U204.7, U204.8
- net at C203.1, R215.1, U202.24 (VDD)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: no longer U203.2, U203.3, U204.2, U204.3
Changed lines of the file:
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@@
 			)
-		)
-		(pin "8"
-		)
-		(pin "6"
-		)
-		(pin "7"
-		)
-		(pin "3"
 		)
 		(pin "1"
@@
 		)
 		(pin "5"
-		)
-		(pin "2"
 		)
 		(instances
@@
 			)
 		)
-		(pin "7"
-		)
 		(pin "1"
-		)
-		(pin "2"
-		)
-		(pin "3"
-		)
-		(pin "6"
 		)
 		(pin "5"
@@
 		(pin "4"
 		)
-		(pin "8"
-		)
 		(instances

Commit message: psu layout
Parts:
- removed R208, R209, R210, R211, R212, R213: 100k, Resistor_SMD:R_0603_1608Metric, symbol Device:R_Small_US
- removed TP201, TP202, TP203, TP204, TP205, TP206: TestPoint, TestPoint:TestPoint_Pad_D1.0mm, symbol Connector:TestPoint
Connections:
- net ALERT: no longer names the net of U202.19 (ALERT)
- net ATTACH: no longer names the net of U202.11 (ATTACH)
- net A_B_SIDE: no longer names the net of U202.17 (A_B_SIDE)
- net GPIO: no longer names the net of U202.15 (GPIO)
- net POWER_OK2: no longer names the net of U202.20 (POWER_OK2)
- net POWER_OK3: no longer names the net of U202.14 (POWER_OK3)
- no-connect marks 5 -> 11
