File: boards/power_supply/pcb/usb_c_pd.kicad_sch (KiCad schematic)
At the start: 34 parts, among them J201 Conn_01x04_Socket, J202 USB4105-GF-A, J203 USB IDC, SW201 PTS526 SK15 SMTR2 LFS, U201 USBLC6-2P6

Commit message: psu layout
Parts:
- renumbered R214 to R208, R215 to R209, R216 to R210, R217 to R211
Changed lines of the file:
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@@
 		(on_board yes)
 		(dnp no)
-		(property "Reference" "R215"
+		(property "Reference" "R209"
 			(at 223.774 45.72 0)
 			(effects
@@
 			(project "power_supply"
 				(path "/6a7d9dc9-f78f-470f-911b-b95256023173/4a384965-6a35-4bf6-849e-cb865e62d5b4"
-					(reference "R215")
+					(reference "R209")
 					(unit 1)
 				)
@@
 		(dnp no)
 		(fields_autoplaced yes)
-		(property "Reference" "R217"
+		(property "Reference" "R211"
 			(at 262.89 64.7699 0)
 			(effects
@@
 			(project "power_supply"
 				(path "/6a7d9dc9-f78f-470f-911b-b95256023173/4a384965-6a35-4bf6-849e-cb865e62d5b4"
-					(reference "R217")
+					(reference "R211")
 					(unit 1)
 				)
@@
 		(on_board yes)
 		(dnp no)
-		(property "Reference" "R216"
+		(property "Reference" "R210"
 			(at 239.522 54.356 90)
 			(effects
@@
 			(project "power_supply"
 				(path "/6a7d9dc9-f78f-470f-911b-b95256023173/4a384965-6a35-4bf6-849e-cb865e62d5b4"
-					(reference "R216")
+					(reference "R210")
 					(unit 1)
 				)
@@
 		(on_board yes)
 		(dnp no)
-		(property "Reference" "R214"
+		(property "Reference" "R208"
 			(at 214.63 57.1499 0)
 			(effects
@@
 			(project "power_supply"
 				(path "/6a7d9dc9-f78f-470f-911b-b95256023173/4a384965-6a35-4bf6-849e-cb865e62d5b4"
-					(reference "R214")
-					(unit 1)
-				)
+					(reference "R208")
+					(unit 1)
+				)
