File: boards/controller/mockup_for_reference_only/mockup/mockup.kicad_sch (KiCad schematic)
At the start: 4 parts, among them SW101 RotaryEncoder_Switch, SW102 RotaryEncoder_Switch, SW103 RotaryEncoder_Switch, U101 CR2013-MI2120

Commit message: controller: Update mockup to use Waveshare display
Signed-off-by: nicholasnloehrke <nicholasnloehrke@gmail.com>
Parts:
- removed SW101, SW102, SW103: RotaryEncoder_Switch, Rotary_Encoder:RotaryEncoder_Alps_EC11E-Switch_Vertical_H20mm, symbol Device:RotaryEncoder_Switch
- removed U101: CR2013-MI2120, Display:CR2013-MI2120, symbol Driver_Display:CR2013-MI2120
