File: boards/controller/pcb/controller.kicad_sch (KiCad schematic)
At the start: 0 parts

Commit message: controller: pcb: Update schematic + layout
Signed-off-by: Nicholas Loehrke <nicholasnloehrke@gmail.com>
Other:
- added sheet Programming/Debug Interface (programming_interface.kicad_sch)
- sheet Bidirectional Load Switch Interface ports: added CH1, CH2, CH3, CH4, CH5, CH6, CH7, CH8, ENn, RSTn; removed PWM1, PWM2, PWM3, PWM4, PWM5, PWM6, PWM7, PWM8
- sheet Charger ports: added ENn, QONn, VBAT_SENSE, VBAT_SENSE_EN; removed none
- sheet Isolated Flyback ports: added 15V+, 15V-; removed none
- sheet LCD Interface ports: added TP_INTn; removed none
- sheet Microcontroller ports: added CHG_QONn, ENC_1SWn, ENC_2SWn, ENC_3SWn, FLYBACK_EN, NRST, PWR_SW_LATCH, PWR_SW_SENSEn, TCP_DBn, TCP_FLTn, TCP_VCC; removed none
- sheet Power Button ports: added MCU_SENSEn; removed none
- sheet USB-C PD ports: added D_N, D_P; removed USB_D_N, USB_D_P
